Commit message: name joints so RViz can subscribe properly

File: urdf/xArm.urdf (robot description, URDF)
Before this commit: robot xArm, 7 links, 6 joints
Joints:
- removed joint joint1
- removed joint joint2
- removed joint joint3
- removed joint joint4
- removed joint joint5
- added joint xArm1: type continuous, parent base_link, child link1, origin xyz=0.0 0.0 0.05 rpy=0.0 0.0 0.0, axis 0 0 1
- added joint xArm2: type continuous, parent link1, child link2, origin xyz=0.0 0.0 0.05 rpy=0.0 0.0 0.0, axis 0 1 0
- added joint xArm3: type continuous, parent link2, child link3, origin xyz=0.0 0.0 0.0965 rpy=0.0 0.0 0.0, axis 0 1 0
- added joint xArm4: type continuous, parent link3, child link4, origin xyz=0.0 0.0 0.0965 rpy=0.0 0.0 0.0, axis 0 1 0
- added joint xArm5: type continuous, parent link4, child link5, origin xyz=0.0 0.0 0.055 rpy=0.0 0.0 0.0, axis 0 0 1

Commit message: added config files to support servo directions

File: urdf/xArm.urdf (robot description, URDF)
Before this commit: robot xArm, 7 links, 6 joints
Joints:
- removed joint xArm1
- removed joint xArm2
- removed joint xArm3
- removed joint xArm4
- removed joint xArm5
- added joint arm1: type continuous, parent base_link, child link1, origin xyz=0.0 0.0 0.05 rpy=0.0 0.0 0.0, axis 0 0 1
- added joint arm2: type continuous, parent link1, child link2, origin xyz=0.0 0.0 0.05 rpy=0.0 0.0 0.0, axis 0 1 0
- added joint arm3: type continuous, parent link2, child link3, origin xyz=0.0 0.0 0.0965 rpy=0.0 0.0 0.0, axis 0 1 0
- added joint arm4: type continuous, parent link3, child link4, origin xyz=0.0 0.0 0.0965 rpy=0.0 0.0 0.0, axis 0 1 0
- added joint arm5: type continuous, parent link4, child link5, origin xyz=0.0 0.0 0.055 rpy=0.0 0.0 0.0, axis 0 0 1

Commit message: added simple shapes (box/cylinder) to urdf file

File: urdf/xArm.urdf (robot description, URDF)
Before this commit: robot xArm, 7 links, 6 joints
Links:
- link link1: geometry visual box size=0.044 0.0285 0.0065; visual box size=0.044 0.0285 0.023
- link link2: geometry visual box size=0.025 0.002 0.045; visual box size=0.025 0.002 0.045
- link link3: geometry visual box size=0.023 0.0285 0.004; visual box size=0.023 0.0285 0.004
- link link4: geometry visual box size=0.025 0.002 0.064; visual box size=0.025 0.002 0.064
Joints:
- joint arm2: origin xyz=0.0 0.0 0.05 rpy=0.0 0.0 0.0 -> xyz=0.0 0.0 0.0425 rpy=0.0 0.0 0.0

Commit message: urdf: added disk for link 5

File: urdf/xArm.urdf (robot description, URDF)
Before this commit: robot xArm, 7 links, 6 joints
Links:
- link link5: geometry visual cylinder length=0.004 radius=0.01
